File: hardware/sadegh_pcb_ready.kicad_sch (KiCad schematic)
At the start: 132 parts, among them J1 Conn_02x04_Odd_Even, P1 Header 8, P3 Header 3, P61 Header 11, Q11A1 2N7000, Q11B1 2N7000, Q11C1 2N7000, Q11D1 2SJ196/BSS92, Q12A1 2N7000, Q12B1 2N7000, Q12C1 2N7000, Q12D1 2SJ196/BSS92, Q13A1 2N7000, Q13B1 2N7000, Q13C1 2N7000, Q13D1 2SJ196/BSS92, Q14A1 2N7000, Q14B1 2N7000, Q14C1 2N7000, Q14D1 2SJ196/BSS92, Q401 2N3904, U1 UART<->USB, U2 W25Q32JVSS, U3 DHT11, U4 AMS1117CD-3.3, U50 LM339J, U51 HCF4051BEY, U52 HCF4051BEY, U61 DSPIC30F4011-30I/P, U71 LM2576D2T-ADJ, U74 LM2576D2T-ADJ, U91 LM2576D2T-ADJ, U92 LM339J, U93 LM339J, U94 LM339J

Commit message: hardware: fix invalid symbol unit name prefixes for KiCad 10
Remove .IntLib and .SchLib suffixes from all lib_symbols names and
their sub-unit definitions (e.g. root_0_SIM900_SIM900.SchLib_1_0 →
root_0_SIM900_SIM900_1_0). KiCad 10 rejects dots in symbol unit name
prefixes. Also update all placed symbol lib_id references to match.

https://claude.ai/code/session_01A9HsvNeuoFeWKhVBvcw39T
Parts:
- C103, C104, C105, C11A1, C11B1, C12A1, C12B1, C13A1, C13B1, C14A1, C14B1, C21, C3, C4, C405, C44, C51, C52, C61, C62, C63, C64, C65, C66, C67, C68, C69, CMMC1, CMMC2: symbol Miscellaneous Devices:root_1_Cap_Miscellaneous Devices.IntLib -> Miscellaneous Devices:root_1_Cap_Miscellaneous Devices
- C401, C403: symbol Miscellaneous Devices:root_0_Cap_Miscellaneous Devices.IntLib -> Miscellaneous Devices:root_0_Cap_Miscellaneous Devices
- C402, C404, Cp101, Cp71, Cp72, Cp73, Cp74, Cp75, Cp91, Cp92: symbol Miscellaneous Devices:root_3_Cap Pol1_Miscellaneous Devices.IntLib_1 -> Miscellaneous Devices:root_3_Cap Pol1_Miscellaneous Devices_1
- D11A1, D12A1, D13A1, D14A1: symbol FSC Discrete Diode:root_1_1N4750A_FSC Discrete Diode.IntLib -> FSC Discrete Diode:root_1_1N4750A_FSC Discrete Diode
- D301, D72, D92: symbol Miscellaneous Devices:root_1_Diode 1N4001_Miscellaneous Devices.IntLib -> Miscellaneous Devices:root_1_Diode 1N4001_Miscellaneous Devices
- D71: symbol Miscellaneous Devices:root_0_mirrored_Diode 1N4007_Miscellaneous Devices.IntLib -> Miscellaneous Devices:root_0_mirrored_Diode 1N4007_Miscellaneous Devices
- D93: symbol Miscellaneous Devices:root_0_Diode 1N4001_Miscellaneous Devices.IntLib -> Miscellaneous Devices:root_0_Diode 1N4001_Miscellaneous Devices
- FBD1, R11A1, R11B1, R11D1, R11E1, R12A1, R12B1, R12D1, R12E1, R13A1, R13B1, R13D1, R13E1, R14A1, R14B1, R14B2, R14D1, R14E1, R301, R302, R303, R304, R61, R903, R904: symbol Miscellaneous Devices:root_1_Res1_Miscellaneous Devices.IntLib -> Miscellaneous Devices:root_1_Res1_Miscellaneous Devices
- L1, L301, L9: symbol Miscellaneous Devices:root_0_Inductor Iron_Miscellaneous Devices.IntLib -> Miscellaneous Devices:root_0_Inductor Iron_Miscellaneous Devices
- MMC1: symbol MMC:root_0_Component_1_MMC.SchLib -> MMC:root_0_Component_1_MMC
- P1: symbol Miscellaneous Connectors:root_0_Header 8_Miscellaneous Connectors.IntLib -> Miscellaneous Connectors:root_0_Header 8_Miscellaneous Connectors
- P3: symbol Miscellaneous Connectors:root_2_Header 3_Miscellaneous Connectors.IntLib -> Miscellaneous Connectors:root_2_Header 3_Miscellaneous Connectors
- P61: symbol Miscellaneous Connectors:root_0_Header 11_Miscellaneous Connectors.IntLib -> Miscellaneous Connectors:root_0_Header 11_Miscellaneous Connectors
- PW1: symbol Miscellaneous Connectors:root_0_Header 4_Miscellaneous Connectors.IntLib -> Miscellaneous Connectors:root_0_Header 4_Miscellaneous Connectors
- Pg1: symbol Miscellaneous Connectors:root_0_SMB_Miscellaneous Connectors.IntLib -> Miscellaneous Connectors:root_0_SMB_Miscellaneous Connectors
- Q11A1, Q11B1, Q11C1, Q12A1, Q12B1, Q12C1, Q13A1, Q13B1, Q13C1, Q14A1, Q14B1, Q14C1: symbol FSC Discrete BJT:root_0_2N3904_FSC Discrete BJT.IntLib -> FSC Discrete BJT:root_0_2N3904_FSC Discrete BJT
- Q11D1, Q12D1, Q13D1, Q14D1: symbol IR Discrete MOSFET - Power:root_2_mirrored_IRF9540N_IR Discrete MOSFET - Power.IntLib -> IR Discrete MOSFET - Power:root_2_mirrored_IRF9540N_IR Discrete MOSFET - Power
- Q401: symbol Miscellaneous Devices:root_0_2N3904_Miscellaneous Devices.IntLib -> Miscellaneous Devices:root_0_2N3904_Miscellaneous Devices
- R11C1, R12C1, R13C1, R14C1, R21, R401, R402, R403, R404, R62, R63, R64, R65: symbol Miscellaneous Devices:root_0_Res1_Miscellaneous Devices.IntLib -> Miscellaneous Devices:root_0_Res1_Miscellaneous Devices
- SIM1: symbol SIMCARD:root_0_Component_1_SIMCARD.SchLib -> SIMCARD:root_0_Component_1_SIMCARD
- SIM900: symbol SIM900:root_0_SIM800A_SIM800A.SchLib -> SIM900:root_0_SIM800A_SIM800A
- U1: symbol FT232RL:root_0_Component_1_FT232RL.SchLib -> FT232RL:root_0_Component_1_FT232RL
- U50, U92, U93, U94: symbol NSC Comparator:root_0_LM339J_NSC Comparator.IntLib -> NSC Comparator:root_0_LM339J_NSC Comparator
- U51, U52: symbol ST Logic Multiplexer:root_0_HCF4051BEY_ST Logic Multiplexer.IntLib -> ST Logic Multiplexer:root_0_HCF4051BEY_ST Logic Multiplexer
- U61: symbol Microchip DSC 16-Bit dsPIC30F:root_0_DSPIC30F4011-30I/P_Microchip DSC 16-Bit dsPIC30F.IntLib -> Microchip DSC 16-Bit dsPIC30F:root_0_DSPIC30F4011-30I/P_Microchip DSC 16-Bit dsPIC30F
- U71, U74, U91: symbol ON Semi Power Mgt Voltage Regulator:root_0_LM2576D2T-ADJ_ON Semi Power Mgt Voltage Regulator.IntLib -> ON Semi Power Mgt Voltage Regulator:root_0_LM2576D2T-ADJ_ON Semi Power Mgt Voltage Regulator
- USB1: symbol USB:root_0_Component_1_USB.SchLib -> USB:root_0_Component_1_USB
Connections:
- net GND: no longer C103.1, C104.1, C105.1, C21.1, C3.1, C4.2, C402.2, C404.2, C405.1, C44.2, C51.1, C52.1, C61.1, C62.1, C63.1, C64.1, C65.1, C66.1, C67.1, C68.2, C69.2, CMMC1.1, CMMC2.1, Cp101.2, Cp74.2
- net VCC: no longer C21.2, C4.1, C51.2, C52.2, C61.2, C62.2, C63.2, C64.2, C67.2, CMMC2.2, Cp74.1
- net VCC-SIM: no longer C404.1, C405.2, L301.2
- net at U61.13 (OSC1/CLKI): no longer C69.1
- net at J1.2 (Pin_2), R14B1.2, U2.3 (~{WP}/IO_{2})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: no longer C3.2, C44.1, CMMC1.2
- net at U1.17 (3V3OUT): no longer C103.2
- net at U61.14 (OSC2/CLKO/RC15): no longer C68.1
- net at R62.1, R63.2, U61.2 (EMUD3/AN0/VREF+/CN2/RB0): no longer C65.2
- net at R64.1, R65.2, U61.3 (EMUC3/AN1/VREF-/CN3/RB1): no longer C66.2
- net at SIM900.25: no longer C402.1
- net at D301.2 (K), U74.2 (OUT): no longer L301.1
- new net: FBD1.2, U1.20 (VCC)
