File: hardware/sadegh_pcb_ready.kicad_sch (KiCad schematic)
At the start: 132 parts, among them J1 Conn_02x04_Odd_Even, P1 Header 8, P3 Header 3, P61 Header 11, Q11A1 2N7000, Q11B1 2N7000, Q11C1 2N7000, Q11D1 2SJ196/BSS92, Q12A1 2N7000, Q12B1 2N7000, Q12C1 2N7000, Q12D1 2SJ196/BSS92, Q13A1 2N7000, Q13B1 2N7000, Q13C1 2N7000, Q13D1 2SJ196/BSS92, Q14A1 2N7000, Q14B1 2N7000, Q14C1 2N7000, Q14D1 2SJ196/BSS92, Q401 2N3904, U1 UART<->USB, U2 W25Q32JVSS, U3 DHT11, U4 AMS1117CD-3.3, U50 LM339J, U51 HCF4051BEY, U52 HCF4051BEY, U61 DSPIC30F4011-30I/P, U71 LM2576D2T-ADJ, U74 LM2576D2T-ADJ, U91 LM2576D2T-ADJ, U92 LM339J, U93 LM339J, U94 LM339J

Commit message: hardware: remove AMS1117, DHT11, and MMC from schematic
Per design requirements:
- Remove AMS1117CD-3.3 voltage regulator (not needed)
- Remove DHT11 temperature/humidity sensor
- Remove MMC/SD card module (replaced by W25Q32 SPI flash)

https://claude.ai/code/session_01A9HsvNeuoFeWKhVBvcw39T
Parts:
- removed MMC1: MMC/SD, Connector_Card:microSD_HC_Molex_104031-0811, symbol MMC:root_0_Component_1_MMC
- removed U3: DHT11, Sensor:Aosong_DHT11_5.5x12.0_P2.54mm, symbol Sensor:DHT11
- removed U4: AMS1117CD-3.3, Package_TO_SOT_SMD:TO-252-3_TabPin2, symbol Regulator_Linear:AMS1117CD-3.3
Changed lines of the file:
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@@
 	)
 	(symbol
-		(lib_id "MMC:root_0_Component_1_MMC")
-		(at 712.47 694.69 0)
-		(unit 1)
-		(exclude_from_sim no)
-		(in_bom yes)
-		(on_board yes)
-		(dnp no)
-		(property "Reference" "MMC1"
-			(at 702.31 684.53 0)
-			(effects
-				(font
-					(size 1.27 1.27)
-				)
-				(justify left bottom)
-			)
-		)
-		(property "Value" "MMC/SD"
-			(at 702.31 704.85 0)
-			(effects
-				(font
-					(size 1.27 1.27)
-				)
-				(justify left bottom)
-			)
-		)
-		(property "Footprint" "Connector_Card:microSD_HC_Molex_104031-0811"
-			(at 712.47 694.69 0)
-			(effects
-				(font
-					(size 1.27 1.27)
-				)
-				(hide yes)
-			)
-		)
-		(property "Datasheet" ""
-			(at 712.47 694.69 0)
-			(effects
-				(font
-					(size 1.27 1.27)
-				)
-				(hide yes)
-			)
-		)
-		(property "Description" ""
-			(at 712.47 694.69 0)
-			(effects
-				(font
-					(size 1.27 1.27)
-				)
-				(hide yes)
-			)
-		)
-		(pin "1"
-		)
-		(pin "2"
-		)
-		(pin "5"
-		)
-		(pin "7"
-		)
-		(pin "4"
-		)
-		(pin "3"
-		)
-		(pin "8"
-		)
-		(pin "6"
-		)
-		(pin "9"
-		)
-		(pin "10"
-		)
-		(instances
-			(project ""
-				(path "/6830c6b4-6be7-4c03-9ee4-6b48bd06f260"
-					(reference "MMC1")
-					(unit 1)
-				)
-			)
-		)
-	)
-	(symbol
 		(lib_id "power:GND")
 		(at 417.83 753.11 0)
@@
 	)
 	(symbol
-		(lib_id "Regulator_Linear:AMS1117CD-3.3")
-		(at 808.99 686.816 180)
-		(unit 1)
-		(exclude_from_sim no)
-		(in_bom yes)
-		(on_board yes)
-		(dnp no)
-		(fields_autoplaced yes)
-		(property "Reference" "U4"
-			(at 808.99 690.626 0)
-			(effects
-				(font
-					(size 1.27 1.27)
-				)
-			)
-		)
-		(property "Value" "AMS1117CD-3.3"
-			(at 808.99 693.166 0)
-			(effects
-				(font
-					(size 1.27 1.27)
-				)
-			)
-		)
-		(property "Footprint" "Package_TO_SOT_SMD:TO-252-3_TabPin2"
-			(at 808.99 691.896 0)
-			(effects
-				(font
-					(size 1.27 1.27)
-				)
-				(hide yes)
-			)
-		)
-		(property "Datasheet" "http://www.advanced-monolithic.com/pdf/ds1117.pdf"
-			(at 806.45 680.466 0)
-			(effects
-				(font
-					(size 1.27 1.27)
-				)
-				(hide yes)
-			)
-		)
-		(property "Description" "1A Low Dropout regulator, positive, 3.3V fixed output, TO-252"
-			(at 808.99 686.816 0)
-			(effects
-				(font
-					(size 1.27 1.27)
-				)
-				(hide yes)
-			)
-		)
-		(pin "2"
-		)
-		(pin "1"
-		)
-		(pin "3"
-		)
-		(instances
-			(project ""
-				(path "/6830c6b4-6be7-4c03-9ee4-6b48bd06f260"
-					(reference "U4")
-					(unit 1)
-				)
-			)
-		)
-	)
-	(symbol
 		(lib_id "power:VCC")
 		(at 760.73 331.47 180)
@@
 					(unit 1)
 				)
-			)
-		)
-	)
-	(symbol
-		(lib_id "Sensor:DHT11")
-		(at 782.32 733.806 0)
-		(unit 1)
-		(exclude_from_sim no)
-		(in_bom yes)
-		(on_board yes)
-		(dnp no)
-		(fields_autoplaced yes)
-		(property "Reference" "U3"
-			(at 775.97 732.5359 0)
-			(effects
-				(font
-					(size 1.27 1.27)
-				)
-				(justify right)
-			)
-		)
-		(property "Value" "DHT11"
-			(at 775.97 735.0759 0)
-			(effects
-				(font
-					(size 1.27 1.27)
-				)
-				(justify right)
-			)
-		)
-		(property "Footprint" "Sensor:Aosong_DHT11_5.5x12.0_P2.54mm"
-			(at 782.32 743.966 0)
-			(effects
-				(font
-					(size 1.27 1.27)
-				)
-				(hide yes)
-			)
-		)
-		(property "Datasheet" "http://akizukidenshi.com/download/ds/aosong/DHT11.pdf"
-			(at 786.13 727.456 0)
-			(effects
-				(font
-					(size 1.27 1.27)
-				)
-				(hide yes)
-			)
-		)
-		(property "Description" "3.3V to 5.5V, temperature and humidity module, DHT11"
-			(at 782.32 733.806 0)
-			(effects
-				(font
-					(size 1.27 1.27)
-				)
-				(hide yes)
-			)
-		)
-		(pin "2"
-		)
-		(pin "3"
-		)
-		(pin "4"
-		)
-		(pin "1"
-		)
-		(instances
-			(project ""
-				(path "/6830c6b4-6be7-4c03-9ee4-6b48bd06f260"
-					(reference "U3")
-					(unit 1)
-				)

Commit message: hardware: fix lib_name sub-unit references after SchLib/IntLib rename
The previous commit fixed sub-unit names in lib_symbols by removing
.IntLib and .SchLib suffixes, but placed symbol instances still referenced
the old names via (lib_name ...) fields. This mismatch would cause KiCad
to fail resolving symbol geometry for capacitors and inductors.

https://claude.ai/code/session_01A9HsvNeuoFeWKhVBvcw39T
Connections:
- net GND: now also C103.1, C104.1, C105.1, C21.1, C3.1, C4.2, C402.2, C404.2, C405.1, C44.2, C51.1, C52.1, C61.1, C62.1, C63.1, C64.1, C65.1, C66.1, C67.1, C68.2, C69.2, CMMC1.1, CMMC2.1, Cp101.2, Cp74.2
- net VCC: now also C21.2, C4.1, C51.2, C52.2, C61.2, C62.2, C63.2, C64.2, C67.2, CMMC2.2, Cp74.1
- net VCC-SIM: now also C404.1, C405.2, L301.2
- net at J1.2 (Pin_2), R14B1.2, U2.3 (~{WP}/IO_{2})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: now also C3.2, C44.1, CMMC1.2
- net at FBD1.2, U1.20 (VCC): now also C104.2, C105.2, Cp101.1
- net at R62.1, R63.2, U61.2 (EMUD3/AN0/VREF+/CN2/RB0): now also C65.2
- net at U61.13 (OSC1/CLKI): now also C69.1
- net at U61.14 (OSC2/CLKO/RC15): now also C68.1
- net at R64.1, R65.2, U61.3 (EMUC3/AN1/VREF-/CN3/RB1): now also C66.2
- net at SIM900.25: now also C402.1
- net at U1.17 (3V3OUT): now also C103.2
- net at D301.2 (K), U74.2 (OUT): now also L301.1
Changed lines of the file:
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@@
 	)
 	(symbol
-		(lib_name "root_1_Cap_Miscellaneous Devices.IntLib_2")
+		(lib_name "root_1_Cap_Miscellaneous Devices_2")
 		(lib_id "Miscellaneous Devices:root_1_Cap_Miscellaneous Devices")
 		(at 308.61 379.73 0)
@@
 	)
 	(symbol
-		(lib_name "root_1_Cap_Miscellaneous Devices.IntLib_1")
+		(lib_name "root_1_Cap_Miscellaneous Devices_1")
 		(lib_id "Miscellaneous Devices:root_1_Cap_Miscellaneous Devices")
 		(at 417.83 95.25 0)
@@
 	)
 	(symbol
-		(lib_name "root_3_Cap Pol1_Miscellaneous Devices.IntLib_1_4")
+		(lib_name "root_3_Cap Pol1_Miscellaneous Devices_1_4")
 		(lib_id "Miscellaneous Devices:root_3_Cap Pol1_Miscellaneous Devices_1")
 		(at 791.21 608.33 0)
@@
 	)
 	(symbol
-		(lib_name "root_1_Cap_Miscellaneous Devices.IntLib_9")
+		(lib_name "root_1_Cap_Miscellaneous Devices_9")
 		(lib_id "Miscellaneous Devices:root_1_Cap_Miscellaneous Devices")
 		(at 158.75 389.89 0)
@@
 	)
 	(symbol
-		(lib_name "root_1_Cap_Miscellaneous Devices.IntLib_16")
+		(lib_name "root_1_Cap_Miscellaneous Devices_16")
 		(lib_id "Miscellaneous Devices:root_1_Cap_Miscellaneous Devices")
 		(at 740.41 692.15 0)
@@
 	)
 	(symbol
-		(lib_name "root_1_Cap_Miscellaneous Devices.IntLib_12")
+		(lib_name "root_1_Cap_Miscellaneous Devices_12")
 		(lib_id "Miscellaneous Devices:root_1_Cap_Miscellaneous Devices")
 		(at 191.77 392.43 0)
@@
 	)
 	(symbol
-		(lib_name "root_1_Cap_Miscellaneous Devices.IntLib_16")
+		(lib_name "root_1_Cap_Miscellaneous Devices_16")
 		(lib_id "Miscellaneous Devices:root_1_Cap_Miscellaneous Devices")
 		(at 703.58 747.776 0)
@@
 	)
 	(symbol
-		(lib_name "root_1_Cap_Miscellaneous Devices.IntLib_11")
+		(lib_name "root_1_Cap_Miscellaneous Devices_11")
 		(lib_id "Miscellaneous Devices:root_1_Cap_Miscellaneous Devices")
 		(at 201.93 392.43 0)
@@
 	)
 	(symbol
-		(lib_name "root_1_Cap_Miscellaneous Devices.IntLib_13")
+		(lib_name "root_1_Cap_Miscellaneous Devices_13")
 		(lib_id "Miscellaneous Devices:root_1_Cap_Miscellaneous Devices")
 		(at 181.61 392.43 0)
@@
 	)
 	(symbol
-		(lib_name "root_3_Cap Pol1_Miscellaneous Devices.IntLib_1_3")
+		(lib_name "root_3_Cap Pol1_Miscellaneous Devices_1_3")
 		(lib_id "Miscellaneous Devices:root_3_Cap Pol1_Miscellaneous Devices_1")
 		(at 290.83 722.63 0)
@@
 	)
 	(symbol
-		(lib_name "root_1_Cap_Miscellaneous Devices.IntLib_6")
+		(lib_name "root_1_Cap_Miscellaneous Devices_6")
 		(lib_id "Miscellaneous Devices:root_1_Cap_Miscellaneous Devices")
 		(at 212.09 392.43 0)
@@
 	)
 	(symbol
-		(lib_name "root_1_Cap_Miscellaneous Devices.IntLib_8")
+		(lib_name "root_1_Cap_Miscellaneous Devices_8")
 		(lib_id "Miscellaneous Devices:root_1_Cap_Miscellaneous Devices")
 		(at 171.45 392.43 0)
@@
 	)
 	(symbol
-		(lib_name "root_1_Cap_Miscellaneous Devices.IntLib_14")
+		(lib_name "root_1_Cap_Miscellaneous Devices_14")
 		(lib_id "Miscellaneous Devices:root_1_Cap_Miscellaneous Devices")
 		(at 877.57 638.81 0)
@@
 	)
 	(symbol
-		(lib_name "root_1_Cap_Miscellaneous Devices.IntLib_14")
+		(lib_name "root_1_Cap_Miscellaneous Devices_14")
 		(lib_id "Miscellaneous Devices:root_1_Cap_Miscellaneous Devices")
 		(at 765.81 732.536 0)
@@
 	)
 	(symbol
-		(lib_name "root_1_Cap_Miscellaneous Devices.IntLib_5")
+		(lib_name "root_1_Cap_Miscellaneous Devices_5")
 		(lib_id "Miscellaneous Devices:root_1_Cap_Miscellaneous Devices")
 		(at 394.97 379.73 0)
@@
 	)
 	(symbol
-		(lib_name "root_1_Cap_Miscellaneous Devices.IntLib_14")
+		(lib_name "root_1_Cap_Miscellaneous Devices_14")
 		(lib_id "Miscellaneous Devices:root_1_Cap_Miscellaneous Devices")
 		(at 792.48 684.276 0)
@@
 	)
 	(symbol
-		(lib_name "root_1_Cap_Miscellaneous Devices.IntLib_15")
+		(lib_name "root_1_Cap_Miscellaneous Devices_15")
 		(lib_id "Miscellaneous Devices:root_1_Cap_Miscellaneous Devices")
 		(at 816.61 610.87 0)
@@
 	)
 	(symbol
-		(lib_name "root_3_Cap Pol1_Miscellaneous Devices.IntLib_1_1")
+		(lib_name "root_3_Cap Pol1_Miscellaneous Devices_1_1")
 		(lib_id "Miscellaneous Devices:root_3_Cap Pol1_Miscellaneous Devices_1")
 		(at 356.87 173.99 0)
@@
 	)
 	(symbol
-		(lib_name "root_1_Cap_Miscellaneous Devices.IntLib_14")
+		(lib_name "root_1_Cap_Miscellaneous Devices_14")
 		(lib_id "Miscellaneous Devices:root_1_Cap_Miscellaneous Devices")
 		(at 819.15 684.276 0)
@@
 	)
 	(symbol
-		(lib_name "root_1_Cap_Miscellaneous Devices.IntLib_10")
+		(lib_name "root_1_Cap_Miscellaneous Devices_10")
 		(lib_id "Miscellaneous Devices:root_1_Cap_Miscellaneous Devices")
 		(at 151.13 392.43 0)
@@
 	)
 	(symbol
-		(lib_name "root_1_Cap_Miscellaneous Devices.IntLib_7")
+		(lib_name "root_1_Cap_Miscellaneous Devices_7")
 		(lib_id "Miscellaneous Devices:root_1_Cap_Miscellaneous Devices")
 		(at 222.25 392.43 0)
@@
 	)
 	(symbol
-		(lib_name "root_1_Cap_Miscellaneous Devices.IntLib_3")
+		(lib_name "root_1_Cap_Miscellaneous Devices_3")
 		(lib_id "Miscellaneous Devices:root_1_Cap_Miscellaneous Devices")
 		(at 435.61 407.67 0)
@@
 	)
 	(symbol
-		(lib_name "root_3_Cap Pol1_Miscellaneous Devices.IntLib_1_2")
+		(lib_name "root_3_Cap Pol1_Miscellaneous Devices_1_2")
 		(lib_id "Miscellaneous Devices:root_3_Cap Pol1_Miscellaneous Devices_1")
 		(at 422.91 120.65 0)
@@
 	)
 	(symbol
-		(lib_name "root_1_Cap_Miscellaneous Devices.IntLib_4")
+		(lib_name "root_1_Cap_Miscellaneous Devices_4")
 		(lib_id "Miscellaneous Devices:root_1_Cap_Miscellaneous Devices")
 		(at 417.83 405.13 0)
@@
 	)
 	(symbol
-		(lib_name "root_1_Cap_Miscellaneous Devices.IntLib_17")
+		(lib_name "root_1_Cap_Miscellaneous Devices_17")
 		(lib_id "Miscellaneous Devices:root_1_Cap_Miscellaneous Devices")
 		(at 806.45 610.87 0)
@@
 	)
 	(symbol
-		(lib_name "root_0_Inductor Iron_Miscellaneous Devices.IntLib_1")
+		(lib_name "root_0_Inductor Iron_Miscellaneous Devices_1")
 		(lib_id "Miscellaneous Devices:root_0_Inductor Iron_Miscellaneous Devices")
 		(at 252.73 572.77 0)
