File: hardware/sadegh_pcb_ready.kicad_sch (KiCad schematic)
At the start: 129 parts, among them J1 Conn_02x04_Odd_Even, P1 Header 8, P3 Header 3, P61 Header 11, Q11A1 2N7000, Q11B1 2N7000, Q11C1 2N7000, Q11D1 2SJ196/BSS92, Q12A1 2N7000, Q12B1 2N7000, Q12C1 2N7000, Q12D1 2SJ196/BSS92, Q13A1 2N7000, Q13B1 2N7000, Q13C1 2N7000, Q13D1 2SJ196/BSS92, Q14A1 2N7000, Q14B1 2N7000, Q14C1 2N7000, Q14D1 2SJ196/BSS92, Q401 2N3904, U1 UART<->USB, U2 W25Q32JVSS, U50 LM339J, U51 HCF4051BEY, U52 HCF4051BEY, U61 DSPIC30F4011-30I/P, U71 LM2576D2T-ADJ, U74 LM2576D2T-ADJ, U91 LM2576D2T-ADJ, U92 LM339J, U93 LM339J, U94 LM339J

Commit message: hardware: fix all footprints to correct THT/DIP packages
Replace SMD/incorrect footprints from Altium import with correct
through-hole (THT) packages matching the actual components used:
- dsPIC30F4011: DIP-40 (was TQFP-44)
- 2N3904: TO-92 THT (was SOT-23 SMD)
- IRF9540N: TO-220-3 THT (was SOT-23 SMD)
- LM339: DIP-14 THT (was SOIC-14 SMD)
- HCF4051: DIP-16 THT (was SOIC-16 SMD)
- LM2576: TO-220-5 THT (was TO-263 SMD)
- Resistors: axial THT (was 0805 SMD)
- Capacitors: disc/radial THT (was 0805 SMD)
- Diodes: DO-41 THT (was SMA SMD)
- Connectors: 2.54mm pin header THT (was 1mm SMD)
- SMD kept for: W25Q32, FT232RL, SIM800A (no THT alternatives)

https://claude.ai/code/session_01A9HsvNeuoFeWKhVBvcw39T
Parts:
- C103, C104, C105, C11A1, C11B1, C12A1, C12B1, C13A1, C13B1, C14A1, C14B1, C3, C4, C401, C405, C44, C65, C66, C68, C69, CMMC1, CMMC2: footprint Capacitor_SMD:C_0805_2012Metric -> Capacitor_THT:C_Disc_D5.0mm_W2.5mm_P5.00mm
- C21, C51, C52, C61, C62, C63, C67: footprint Capacitor_SMD:C_1206_3216Metric -> Capacitor_THT:C_Disc_D5.0mm_W2.5mm_P5.00mm
- C402, Cp101: footprint Capacitor_SMD:CP_Elec_5x5.3 -> Capacitor_THT:CP_Radial_D8.0mm_P3.50mm
- C403: footprint Capacitor_SMD:CP_Elec_6.3x5.4 -> Capacitor_THT:C_Disc_D5.0mm_W2.5mm_P5.00mm
- C404: footprint Capacitor_SMD:CP_Elec_10x10 -> Capacitor_THT:CP_Radial_D8.0mm_P3.50mm
- C64: footprint CAPR2.54-4x2.5 -> Capacitor_THT:C_Disc_D5.0mm_W2.5mm_P5.00mm
- Cp71, Cp72, Cp73, Cp74, Cp75, Cp91, Cp92: footprint Capacitor_SMD:CP_Elec_10x12.5 -> Capacitor_THT:CP_Radial_D8.0mm_P3.50mm
- D11A1, D12A1, D13A1, D14A1, D301, D71, D92, D93: footprint Diode_SMD:D_SMA -> Diode_THT:D_DO-41_SOD81_P10.16mm_Horizontal
- D72: footprint DO-41 -> Diode_THT:D_DO-41_SOD81_P10.16mm_Horizontal
- FBD1, R11A1, R11B1, R11C1, R11D1, R11E1, R12A1, R12B1, R12C1, R12D1, R12E1, R13A1, R13B1, R13D1, R13E1, R14A1, R14B1, R14B2, R14C1, R14D1, R14E1, R301, R302, R303, R401, R402, R403, R404, R61, R62, R63, R64, R65, R903, R904: footprint Resistor_SMD:R_0805_2012Metric -> Resistor_THT:R_Axial_DIN0207_L6.3mm_D2.5mm_P10.16mm_Horizontal
- J1: footprint Connector_PinHeader_1.00mm:PinHeader_2x04_P1.00mm_Vertical_SMD -> Connector_PinHeader_2.54mm:PinHeader_2x04_P2.54mm_Vertical
- L1, L301, L9: footprint Inductor_SMD:L_12x12mm_H8mm -> Inductor_THT:L_Radial_D8.7mm_P5.00mm
- P1: footprint Connector_Phoenix_GMSTB:PhoenixContact_GMSTBA_2,5_8-G_1x08_P7.50mm_Horizontal -> Connector_PinHeader_2.54mm:PinHeader_1x08_P2.54mm_Vertical
- P3: footprint Connector_PinHeader_1.00mm:PinHeader_1x03_P1.00mm_Vertical_SMD_Pin1Left -> Connector_PinHeader_2.54mm:PinHeader_1x03_P2.54mm_Vertical
- P61: footprint Connector_PinHeader_1.00mm:PinHeader_1x11_P1.00mm_Vertical_SMD_Pin1Left -> Connector_PinHeader_2.54mm:PinHeader_1x11_P2.54mm_Vertical
- PW1: footprint Connector_Phoenix_GMSTB:PhoenixContact_GMSTBA_2,5_4-G_1x04_P7.50mm_Horizontal -> Connector_PinHeader_2.54mm:PinHeader_1x04_P2.54mm_Vertical
- Q11A1, Q11B1, Q11C1, Q12A1, Q12B1, Q12C1, Q13A1, Q13B1, Q13C1, Q14A1, Q14B1, Q14C1, Q401: footprint Package_TO_SOT_SMD:SOT-23 -> Package_TO_SOT_THT:TO-92_Inline
- Q11D1, Q12D1, Q13D1, Q14D1: footprint Package_TO_SOT_SMD:SOT-23 -> Package_TO_SOT_THT:TO-220-3_Vertical
- R13C1, R21, R304: footprint AXIAL-0.3 -> Resistor_THT:R_Axial_DIN0207_L6.3mm_D2.5mm_P10.16mm_Horizontal
- U50, U92, U93, U94: footprint Package_SO:SOIC-14_3.9x8.7mm_P1.27mm -> Package_DIP:DIP-14_W7.62mm
- U51, U52: footprint Package_SO:SOIC-16_3.9x9.9mm_P1.27mm -> Package_DIP:DIP-16_W7.62mm
- U61: footprint Package_QFP:TQFP-44_10x10mm_P0.8mm -> Package_DIP:DIP-40_W15.24mm
- U71, U74, U91: footprint Package_TO_SOT_SMD:TO-263-5_TabPin3 -> Package_TO_SOT_THT:TO-220-5_P3.4mm_Vertical

Commit message: hardware: fix ERC errors - convert hierarchical labels to global labels
- Convert all 43 hierarchical_label to global_label (Altium import
  artifact; this is a flat single-sheet schematic with no hierarchy)
- Remove orphaned labels for removed components: RTCCS (RTC removed),
  MMCINT and MMCCS (MMC removed)

Fixes: "hierarchical label cannot be connected to non-existent parent
sheet" errors in KiCad ERC.

https://claude.ai/code/session_01A9HsvNeuoFeWKhVBvcw39T
Connections:
- net MMCCS: no longer names the net of U2.1 (~{CS})
- net MMCCS: no longer U61.29 (C1TX/RF1)
- net MMCINT: no longer names the net of R21.1, U61.17 (~{FLTA}/INT0/RE8)
- net RTCCS: no longer names the net of U61.30 (C1RX/RF0)
Changed lines of the file:
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@@
 		)
 	)
-	(hierarchical_label "MISO"
+	(global_label "MISO"
 		(shape output)
 		(at 694.69 699.77 180)
@@
 		)
 	)
-	(hierarchical_label "MOSI"
+	(global_label "MOSI"
 		(shape input)
 		(at 671.83 697.23 180)
@@
 		)
 	)
-	(hierarchical_label "RTCCS"
-		(shape output)
-		(at 318.77 448.31 180)
-		(effects
-			(font
-				(size 1.27 1.27)
-			)
-			(justify right)
-		)
-	)
-	(hierarchical_label "SCK"
+	(global_label "SCK"
 		(shape input)
 		(at 293.37 463.55 180)
@@
 		)
 	)
-	(hierarchical_label "PWRKEY"
+	(global_label "PWRKEY"
 		(shape input)
 		(at 269.24 118.11 180)
@@
 		)
 	)
-	(hierarchical_label "mmcerror"
+	(global_label "mmcerror"
 		(shape output)
 		(at 504.19 519.43 180)
@@
 		)
 	)
-	(hierarchical_label "mmcerror"
+	(global_label "mmcerror"
 		(shape output)
 		(at 407.67 412.75 180)
@@
 		)
 	)
-	(hierarchical_label "SIMONOFF"
+	(global_label "SIMONOFF"
 		(shape passive)
 		(at 410.21 405.13 180)
@@
 		)
 	)
-	(hierarchical_label "MDMSTAT"
+	(global_label "MDMSTAT"
 		(shape output)
 		(at 331.47 85.09 180)
@@
 		)
 	)
-	(hierarchical_label "MMCCS"
-		(shape input)
-		(at 651.51 692.15 180)
-		(effects
-			(font
-				(size 1.27 1.27)
-			)
-			(justify right)
-		)
-	)
-	(hierarchical_label "SIM900_TXD"
+	(global_label "SIM900_TXD"
 		(shape output)
 		(at 283.21 458.47 0)
@@
 		)
 	)
-	(hierarchical_label "SIM900_RXD"
+	(global_label "SIM900_RXD"
 		(shape input)
 		(at 247.65 461.01 0)
@@
 		)
 	)
-	(hierarchical_label "FT232RL_TXD"
+	(global_label "FT232RL_TXD"
 		(shape output)
 		(at 946.15 600.71 0)
@@
 		)
 	)
-	(hierarchical_label "MOSI"
+	(global_label "MOSI"
 		(shape input)
 		(at 293.37 455.93 180)
@@
 		)
 	)
-	(hierarchical_label "loopselB"
+	(global_label "loopselB"
 		(shape passive)
 		(at 532.13 265.43 180)
@@
 		)
 	)
-	(hierarchical_label "loopselB"
+	(global_label "loopselB"
 		(shape passive)
 		(at 407.67 438.15 180)
@@
 		)
 	)
-	(hierarchical_label "CAPTURE"
+	(global_label "CAPTURE"
 		(shape passive)
 		(at 405.13 267.97 180)
@@
 		)
 	)
-	(hierarchical_label "PWRKEY"
+	(global_label "PWRKEY"
 		(shape input)
 		(at 407.67 417.83 180)
@@
 		)
 	)
-	(hierarchical_label "SIM900_RXD"
+	(global_label "SIM900_RXD"
 		(shape input)
 		(at 313.69 133.35 180)
@@
 		)
 	)
-	(hierarchical_label "SCK"
+	(global_label "SCK"
 		(shape input)
 		(at 661.67 694.69 180)
@@
 		)
 	)
-	(hierarchical_label "MISO"
+	(global_label "MISO"
 		(shape output)
 		(at 313.69 453.39 180)
@@
 		)
 	)
-	(hierarchical_label "MDMSTAT"
+	(global_label "MDMSTAT"
 		(shape output)
 		(at 407.67 415.29 180)
@@
 		)
 	)
-	(hierarchical_label "loopselB"
+	(global_label "loopselB"
 		(shape passive)
 		(at 410.21 260.35 180)
@@
 		)
 	)
-	(hierarchical_label "MMCCS"
-		(shape output)
-		(at 318.77 450.85 180)
-		(effects
-			(font
-				(size 1.27 1.27)
-			)
-			(justify right)
-		)
-	)
-	(hierarchical_label "FT232RL_RXD"
+	(global_label "FT232RL_RXD"
 		(shape input)
 		(at 946.15 603.25 0)
@@
 		)
 	)
-	(hierarchical_label "MOSI"
+	(global_label "MOSI"
 		(shape input)
 		(at 668.02 731.266 180)
@@
 		)
 	)
-	(hierarchical_label "loopselC"
+	(global_label "loopselC"
 		(shape passive)
 		(at 532.13 267.97 180)
@@
 		)
 	)
-	(hierarchical_label "FT232RL_TXD"
+	(global_label "FT232RL_TXD"
 		(shape output)
 		(at 410.21 427.99 180)
@@
 		)
 	)
-	(hierarchical_label "loopselA"
+	(global_label "loopselA"
 		(shape passive)
 		(at 407.67 435.61 180)
@@
 		)
 	)
-	(hierarchical_label "SCK"
+	(global_label "SCK"
 		(shape input)
 		(at 657.86 728.726 180)
@@
 		)
 	)
-	(hierarchical_label "MMCCS"
-		(shape input)
-		(at 647.7 726.186 180)
-		(effects
-			(font
-				(size 1.27 1.27)
-			)
-			(justify right)
-		)
-	)
-	(hierarchical_label "MMCINT"
-		(shape output)
-		(at 461.01 458.47 180)
-		(effects
-			(font
-				(size 1.27 1.27)
-			)
-			(justify right)
-		)
-	)
-	(hierarchical_label "loopselA"
+	(global_label "loopselA"
 		(shape passive)
 		(at 532.13 262.89 180)
@@
 		)
 	)
-	(hierarchical_label "MISO"
+	(global_label "MISO"
 		(shape output)
 		(at 681.99 733.806 180)
@@
 		)
 	)
-	(hierarchical_label "loopselC"
+	(global_label "loopselC"
 		(shape passive)
 		(at 410.21 262.89 180)
@@
 		)
 	)
-	(hierarchical_label "loopselA"
+	(global_label "loopselA"
 		(shape passive)
 		(at 410.21 257.81 180)
@@
 		)
 	)
-	(hierarchical_label "NetLight"
+	(global_label "NetLight"
 		(shape output)
 		(at 433.07 82.55 0)
@@
 		)
 	)
-	(hierarchical_label "NetLight"
+	(global_label "NetLight"
 		(shape output)
 		(at 504.19 516.89 180)
@@
 		)
 	)
-	(hierarchical_label "SIM900_TXD"
+	(global_label "SIM900_TXD"
 		(shape output)
 		(at 313.69 130.81 180)
@@
 		)
 	)
-	(hierarchical_label "SIMONOFF"
+	(global_label "SIMONOFF"
 		(shape passive)
 		(at 204.47 577.85 180)
@@
 		)
 	)
-	(hierarchical_label "CAPTURE"
+	(global_label "CAPTURE"
 		(shape passive)
 		(at 407.67 410.21 180)
@@
 		)
 	)
-	(hierarchical_label "FT232RL_RXD"
+	(global_label "FT232RL_RXD"
 		(shape input)
 		(at 410.21 425.45 180)
@@
 		)
 	)
-	(hierarchical_label "loopselC"
+	(global_label "loopselC"
 		(shape passive)
 		(at 407.67 440.69 180)

Commit message: hardware: fix 4 footprints to use available library variants
- LM2576: TO-220-5_P3.4mm_Vertical -> TO-220-5_Vertical (available)
- Inductor: L_Radial_D8.7mm_P5.00mm -> Fastron_07HCP variant (available)
- SIM800A: SIMCom_SIM800 -> SIMCom_SIM800C (available in RF_GSM)
- W25Q32: SOIC-8_5.3x5.3mm -> SOIC-8W_5.3x5.3mm (wide body, available)

All 22 footprints now confirmed present in KiCad standard library.

https://claude.ai/code/session_01A9HsvNeuoFeWKhVBvcw39T
Parts:
- L1, L301, L9: footprint Inductor_THT:L_Radial_D8.7mm_P5.00mm -> Inductor_THT:L_Radial_D8.7mm_P5.00mm_Fastron_07HCP
- SIM900: footprint RF_GSM:SIMCom_SIM800 -> RF_GSM:SIMCom_SIM800C
- U2: footprint Package_SO:SOIC-8_5.3x5.3mm_P1.27mm -> Package_SO:SOIC-8W_5.3x5.3mm_P1.27mm
- U71, U74, U91: footprint Package_TO_SOT_THT:TO-220-5_P3.4mm_Vertical -> Package_TO_SOT_THT:TO-220-5_Vertical
Changed lines of the file:
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@@
 			)
 		)
-		(property "Footprint" "Package_TO_SOT_THT:TO-220-5_P3.4mm_Vertical"
+		(property "Footprint" "Package_TO_SOT_THT:TO-220-5_Vertical"
 			(at 212.09 712.47 0)
 			(effects
@@
 			)
 		)
-		(property "Footprint" "Package_SO:SOIC-8_5.3x5.3mm_P1.27mm"
+		(property "Footprint" "Package_SO:SOIC-8W_5.3x5.3mm_P1.27mm"
 			(at 723.9 732.536 0)
 			(effects
@@
 			)
 		)
-		(property "Footprint" "Inductor_THT:L_Radial_D8.7mm_P5.00mm"
+		(property "Footprint" "Inductor_THT:L_Radial_D8.7mm_P5.00mm_Fastron_07HCP"
 			(at 433.07 715.01 0)
 			(effects
@@
 			)
 		)
-		(property "Footprint" "Inductor_THT:L_Radial_D8.7mm_P5.00mm"
+		(property "Footprint" "Inductor_THT:L_Radial_D8.7mm_P5.00mm_Fastron_07HCP"
 			(at 252.73 715.01 0)
 			(effects
@@
 			)
 		)
-		(property "Footprint" "Package_TO_SOT_THT:TO-220-5_P3.4mm_Vertical"
+		(property "Footprint" "Package_TO_SOT_THT:TO-220-5_Vertical"
 			(at 392.43 712.47 0)
 			(effects
@@
 			)
 		)
-		(property "Footprint" "RF_GSM:SIMCom_SIM800"
+		(property "Footprint" "RF_GSM:SIMCom_SIM800C"
 			(at 356.87 130.81 0)
 			(effects
@@
 			)
 		)
-		(property "Footprint" "Package_TO_SOT_THT:TO-220-5_P3.4mm_Vertical"
+		(property "Footprint" "Package_TO_SOT_THT:TO-220-5_Vertical"
 			(at 209.55 572.77 0)
 			(effects
@@
 			)
 		)
-		(property "Footprint" "Inductor_THT:L_Radial_D8.7mm_P5.00mm"
+		(property "Footprint" "Inductor_THT:L_Radial_D8.7mm_P5.00mm_Fastron_07HCP"
 			(at 252.73 572.77 0)
 			(effects

Commit message: hardware: convert all footprints to SMD and fix remaining PCB update errors
- Convert all THT/DIP footprints to SMD equivalents:
  - Resistors: R_Axial → R_0805_2012Metric (38 parts)
  - Caps disc: C_Disc → C_0805_2012Metric (31 parts)
  - Caps electrolytic: CP_Radial → C_Tantalum_E_7.3x4.3mm (10 parts)
  - Transistors: TO-92 → SOT-23 (13 parts)
  - MOSFETs: TO-220-3 → TO-263-3_TabPin2 (4 parts)
  - LM2576: TO-220-5 → TO-263-5_TabPin6 (3 parts, tab=pin6)
  - DIP-14 → SOIC-14 (4 LM339)
  - DIP-16 → SOIC-16 (2 HCF4051)
  - DIP-40 dsPIC → TQFP-44_10x10mm (1 part)
  - Inductors: L_Radial → L_12x12mm_H8mm (3 parts)
  - W25Q32: SOIC-8W → SOIC-8_3.9x4.9mm_P1.27mm (2 parts)
  - SIM800A: SIMCom_SIM800C → SIMCom_SIM900 (68 pads match symbol)
- Fix SIM1: create custom 8-pin microSIM footprint with switch pads (4,8)
- Fix USB1: change to USB_Micro-B footprint with 6 pads matching symbol
- Add fp-lib-table for project-local custom_footprints library
- Add custom_footprints.pretty directory with microSIM_JAE_SF53S006_8pin

https://claude.ai/code/session_01A9HsvNeuoFeWKhVBvcw39T
Parts:
- C103, C104, C105, C11A1, C11B1, C12A1, C12B1, C13A1, C13B1, C14A1, C14B1, C21, C3, C4, C401, C403, C405, C44, C51, C52, C61, C62, C63, C64, C65, C66, C67, C68, C69, CMMC1, CMMC2: footprint Capacitor_THT:C_Disc_D5.0mm_W2.5mm_P5.00mm -> Capacitor_SMD:C_0805_2012Metric
- C402, C404, Cp101, Cp71, Cp72, Cp73, Cp74, Cp75, Cp91, Cp92: footprint Capacitor_THT:CP_Radial_D8.0mm_P3.50mm -> Capacitor_SMD:C_Tantalum_E_7.3x4.3mm_P4.10mm
- FBD1, R11A1, R11B1, R11C1, R11D1, R11E1, R12A1, R12B1, R12C1, R12D1, R12E1, R13A1, R13B1, R13C1, R13D1, R13E1, R14A1, R14B1, R14B2, R14C1, R14D1, R14E1, R21, R301, R302, R303, R304, R401, R402, R403, R404, R61, R62, R63, R64, R65, R903, R904: footprint Resistor_THT:R_Axial_DIN0207_L6.3mm_D2.5mm_P10.16mm_Horizontal -> Resistor_SMD:R_0805_2012Metric
- L1, L301, L9: footprint Inductor_THT:L_Radial_D8.7mm_P5.00mm_Fastron_07HCP -> Inductor_SMD:L_12x12mm_H8mm
- Q11A1, Q11B1, Q11C1, Q12A1, Q12B1, Q12C1, Q13A1, Q13B1, Q13C1, Q14A1, Q14B1, Q14C1, Q401: footprint Package_TO_SOT_THT:TO-92_Inline -> Package_TO_SOT_SMD:SOT-23
- Q11D1, Q12D1, Q13D1, Q14D1: footprint Package_TO_SOT_THT:TO-220-3_Vertical -> Package_TO_SOT_SMD:TO-263-3_TabPin2
- SIM1: footprint Connector_Card:microSIM_JAE_SF53S006VCBR2000 -> custom_footprints:microSIM_JAE_SF53S006_8pin
- SIM900: footprint RF_GSM:SIMCom_SIM800C -> RF_GSM:SIMCom_SIM900
- U2: footprint Package_SO:SOIC-8W_5.3x5.3mm_P1.27mm -> Package_SO:SOIC-8_3.9x4.9mm_P1.27mm
- U50, U92, U93, U94: footprint Package_DIP:DIP-14_W7.62mm -> Package_SO:SOIC-14_3.9x8.7mm_P1.27mm
- U51, U52: footprint Package_DIP:DIP-16_W7.62mm -> Package_SO:SOIC-16_3.9x9.9mm_P1.27mm
- U61: footprint Package_DIP:DIP-40_W15.24mm -> Package_QFP:TQFP-44_10x10mm_P0.8mm
- U71, U74, U91: footprint Package_TO_SOT_THT:TO-220-5_Vertical -> Package_TO_SOT_SMD:TO-263-5_TabPin6
- USB1: footprint Connector_USB:USB_B_Lumberg_2411_02_Horizontal -> Connector_USB:USB_Micro-B_Amphenol_10103594-0001LF_Horizontal

Commit message: hardware: replace 2SJ196/BSS92 with SI2309DS, add Phoenix connectors, add ICSP header
- Replace 2SJ196/BSS92 P-channel MOSFET with SI2309DS (SOT-23):
  - 4 instances updated (Value + Footprint)
  - Custom SOT-23_GDS footprint: pad2=Drain(physical pin3), pad3=Source(physical pin2)
    to match the schematic symbol pin assignment G=1, D=2, S=3
- P1 (8-pin signal connector): PinHeader_1x08 → Phoenix Contact MSTB_2,5_8-GF-5,08
  (5.08mm pitch, accepts up to 2.5mm² wire, threaded flange for strain relief)
- PW1 (4-pin power input): PinHeader_1x04 → Phoenix Contact MSTB_2,5_4-GF-5,08
  (5.08mm pitch, accepts 0.2-2.5mm² wire - suitable for 1-2mm² power wiring)
- Add ICSP1 programming header (PICkit3):
  - 6-pin 2.54mm vertical header (Connector_PinHeader_2.54mm:PinHeader_1x06)
  - Pin 1: MCLR/VPP
  - Pin 2: VDD target (+3.3V)
  - Pin 3: GND
  - Pin 4: PGD = MOSI (RF3/pin25 of dsPIC30F4011)
  - Pin 5: PGC = MISO (RF2/pin26 of dsPIC30F4011)
  - Pin 6: NC/AUX

https://claude.ai/code/session_01A9HsvNeuoFeWKhVBvcw39T
Parts:
- P1: value Header 8 -> Phoenix_MSTB_8pin_5.08mm; footprint Connector_PinHeader_2.54mm:PinHeader_1x08_P2.54mm_Vertical -> Connector_Phoenix_MSTB:PhoenixContact_MSTB_2,5_8-GF-5,08_1x08_P5.08mm_Horizontal_ThreadedFlange
- PW1: value Header 4 -> Phoenix_MSTB_4pin_5.08mm; footprint Connector_PinHeader_2.54mm:PinHeader_1x04_P2.54mm_Vertical -> Connector_Phoenix_MSTB:PhoenixContact_MSTB_2,5_4-GF-5,08_1x04_P5.08mm_Horizontal_ThreadedFlange
- Q11D1, Q12D1, Q13D1, Q14D1: value 2SJ196/BSS92 -> SI2309DS; footprint Package_TO_SOT_SMD:TO-263-3_TabPin2 -> custom_footprints:SOT-23_GDS
Changed lines of the file:
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@@
 			)
 		)
-		(property "Value" "2SJ196/BSS92"
+		(property "Value" "SI2309DS"
 			(at 756.666 404.876 0)
 			(effects
@@
 			)
 		)
-		(property "Footprint" "Package_TO_SOT_SMD:TO-263-3_TabPin2"
+		(property "Footprint" "custom_footprints:SOT-23_GDS"
 			(at 748.03 405.13 0)
 			(effects
@@
 			)
 		)
-		(property "Value" "Header 8"
+		(property "Value" "Phoenix_MSTB_8pin_5.08mm"
 			(at 910.59 328.93 0)
 			(effects
@@
 			)
 		)
-		(property "Footprint" "Connector_PinHeader_2.54mm:PinHeader_1x08_P2.54mm_Vertical"
+		(property "Footprint" "Connector_Phoenix_MSTB:PhoenixContact_MSTB_2,5_8-GF-5,08_1x08_P5.08mm_Horizontal_ThreadedFlange"
 			(at 910.59 303.53 0)
 			(effects
@@
 			)
 		)
-		(property "Value" "2SJ196/BSS92"
+		(property "Value" "SI2309DS"
 			(at 766.826 227.076 0)
 			(effects
@@
 			)
 		)
-		(property "Footprint" "Package_TO_SOT_SMD:TO-263-3_TabPin2"
+		(property "Footprint" "custom_footprints:SOT-23_GDS"
 			(at 758.19 227.33 0)
 			(effects
@@
 			)
 		)
-		(property "Value" "Header 4"
+		(property "Value" "Phoenix_MSTB_4pin_5.08mm"
 			(at 214.63 504.19 0)
 			(effects
@@
 			)
 		)
-		(property "Footprint" "Connector_PinHeader_2.54mm:PinHeader_1x04_P2.54mm_Vertical"
+		(property "Footprint" "Connector_Phoenix_MSTB:PhoenixContact_MSTB_2,5_4-GF-5,08_1x04_P5.08mm_Horizontal_ThreadedFlange"
 			(at 214.63 488.95 0)
 			(effects
@@
 			)
 		)
-		(property "Value" "2SJ196/BSS92"
+		(property "Value" "SI2309DS"
 			(at 764.286 290.576 0)
 			(effects
@@
 			)
 		)
-		(property "Footprint" "Package_TO_SOT_SMD:TO-263-3_TabPin2"
+		(property "Footprint" "custom_footprints:SOT-23_GDS"
 			(at 755.65 290.83 0)
 			(effects
@@
 			)
 		)
-		(property "Value" "2SJ196/BSS92"
+		(property "Value" "SI2309DS"
 			(at 764.286 341.376 0)
 			(effects
@@
 			)
 		)
-		(property "Footprint" "Package_TO_SOT_SMD:TO-263-3_TabPin2"
+		(property "Footprint" "custom_footprints:SOT-23_GDS"
 			(at 755.65 341.63 0)
 			(effects
@@
 	(embedded_fonts no)
 )
+	(symbol "custom:ICSP_Header6"
+			(pin_numbers
+				(hide yes)
+			)
+			(exclude_from_sim no)
+			(in_bom yes)
+			(on_board yes)
+			(property "Reference" ""
+				(at 0 0 0)
+				(effects
+					(font
+						(size 1.27 1.27)
+					)
+				)
+			)
+			(property "Value" ""
+				(at 0 0 0)
+				(effects
+					(font
+						(size 1.27 1.27)
+					)
+				)
+			)
+			(property "Footprint" ""
+				(at 0 0 0)
+				(effects
+					(font
+						(size 1.27 1.27)
+					)
+					(hide yes)
+				)
+			)
+			(property "Datasheet" ""
+				(at 0 0 0)
+				(effects
+					(font
+						(size 1.27 1.27)
+					)
+					(hide yes)
+				)
+			)
+			(property "Description" "6-pin ICSP/PICkit3 programming header"
+				(at 0 0 0)
+				(effects
+					(font
+						(size 1.27 1.27)
+					)
+					(hide yes)
+				)
+			)
+			(symbol "ICSP_Header6_1_0"
+				(rectangle
+					(start 7.62 0)
+					(end 0 -17.78)
+					(stroke
+						(width 0.0254)
+						(type solid)
+						(color 128 0 0 1)
+					)
+					(fill
+						(type background)
+					)
+				)
+				(pin passive line
+					(at -5.08 -2.54 0)
+					(length 5.08)
+					(name "MCLR"
+						(effects (font (size 1.27 1.27)))
+					)
+					(number "1"
+						(effects (font (size 1.27 1.27)))
+					)
+				)
+				(pin passive line
+					(at -5.08 -5.08 0)
+					(length 5.08)
+					(name "VDD"
+						(effects (font (size 1.27 1.27)))
+					)
+					(number "2"
+						(effects (font (size 1.27 1.27)))
+					)
+				)
+				(pin passive line
+					(at -5.08 -7.62 0)
+					(length 5.08)
+					(name "GND"
+						(effects (font (size 1.27 1.27)))
+					)
+					(number "3"
+						(effects (font (size 1.27 1.27)))
+					)
+				)
+				(pin passive line
+					(at -5.08 -10.16 0)
+					(length 5.08)
+					(name "PGD"
+						(effects (font (size 1.27 1.27)))
+					)
+					(number "4"
+						(effects (font (size 1.27 1.27)))
+					)
+				)
+				(pin passive line
+					(at -5.08 -12.7 0)
+					(length 5.08)
+					(name "PGC"
+						(effects (font (size 1.27 1.27)))
+					)
+					(number "5"
+						(effects (font (size 1.27 1.27)))
+					)
+				)
+				(pin passive line
+					(at -5.08 -15.24 0)
+					(length 5.08)
+					(name "NC"
+						(effects (font (size 1.27 1.27)))
+					)
+					(number "6"
+						(effects (font (size 1.27 1.27)))
+					)
+				)
+			)
+			(embedded_fonts
+	(symbol
+		(lib_id "custom:ICSP_Header6")
+		(at 920.0 450.0 0)
+		(unit 1)
+		(exclude_from_sim no)
+		(in_bom yes)
+		(on_board yes)
+		(dnp no)
+		(property "Reference" "ICSP1"
+			(at 920.0 445.0 0)
+			(effects
+				(font
+					(size 1.27 1.27)
+				)
+				(justify left bottom)
+			)
+		)
+		(property "Value" "PICkit3_ICSP"
+			(at 920.0 470.0 0)
+			(effects
+				(font
+					(size 1.27 1.27)
+				)
+				(justify left bottom)
+			)
+		)
+		(property "Footprint" "Connector_PinHeader_2.54mm:PinHeader_1x06_P2.54mm_Vertical"
+			(at 920.0 450.0 0)
+			(effects
+				(font
+					(size 1.27 1.27)
+				)
+				(hide yes)
+			)
+		)
+		(property "Datasheet" ""
+			(at 920.0 450.0 0)
+			(effects
+				(font
+					(size 1.27 1.27)
+				)
+				(hide yes)
+			)
+		)
+		(property "Description" "PICkit3 ICSP Programming Header 6-pin 2.54mm"
+			(at 920.0 450.0 0)
+			(effects
+				(font
+					(size 1.27 1.27)
+				)
+				(hide yes)
+			)
+		)
+		(pin "1"
+		)
+		(pin "2"
+		)
+		(pin "3"
+		)
+		(pin "4"
+		)
+		(pin "5"
+		)
+		(pin "6"
+		)
+		(instances
+			(project ""
+				(path "/6830c6b4-6be7-4c03-9ee4-6b48bd06f260"
+					(reference "ICSP1")
+					(unit 1)
+				)
+			)
+		)
+	)
+ no)
+		)
