File: hardware/sadegh_pcb_ready.kicad_sch (KiCad schematic)
At the start: 129 parts, among them J1 Conn_02x04_Odd_Even, P1 Phoenix_MSTB_8pin_5.08mm, P3 Header 3, P61 Header 11, Q11A1 2N7000, Q11B1 2N7000, Q11C1 2N7000, Q11D1 SI2309DS, Q12A1 2N7000, Q12B1 2N7000, Q12C1 2N7000, Q12D1 SI2309DS, Q13A1 2N7000, Q13B1 2N7000, Q13C1 2N7000, Q13D1 SI2309DS, Q14A1 2N7000, Q14B1 2N7000, Q14C1 2N7000, Q14D1 SI2309DS, Q401 2N3904, U1 UART<->USB, U2 W25Q32JVSS, U50 LM339J, U51 HCF4051BEY, U52 HCF4051BEY, U61 DSPIC30F4011-30I/P, U71 LM2576D2T-ADJ, U74 LM2576D2T-ADJ, U91 LM2576D2T-ADJ, U92 LM339J, U93 LM339J, U94 LM339J

Commit message: hardware: fix LM339J multi-unit reference - merge 4 ICs into 1
The 4 LM339J comparator units were imported from Altium with separate
references (U50, U92, U93, U94), causing 4 physical ICs to appear on
the PCB instead of 1. All units are now under the same reference U50:

  U50 (unit 1) - Comparator 1: IN1+, IN1-, OUT1 (pins 4,5,2)
  U50 (unit 2) - Comparator 2: IN2+, IN2-, OUT2 (pins 6,7,1)
  U50 (unit 3) - Comparator 3: IN3+, IN3-, OUT3 (pins 8,9,14)
  U50 (unit 4) - Comparator 4: IN4+, IN4-, OUT4 (pins 10,11,13)

Power pins V+ (pin 3) and GND (pin 12) are present in each unit
instance per the Altium import convention. PCB will now show 1x
SOIC-14 footprint instead of 4x.

https://claude.ai/code/session_01A9HsvNeuoFeWKhVBvcw39T
Parts:
- renumbered U92 to U50, U93 to U50, U94 to U50
Changed lines of the file:
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@@
 		(on_board yes)
 		(dnp no)
-		(property "Reference" "U92"
+		(property "Reference" "U50"
 			(at 900.938 422.656 0)
 			(effects
@@
 			(project ""
 				(path "/6830c6b4-6be7-4c03-9ee4-6b48bd06f260"
-					(reference "U92")
+					(reference "U50")
 					(unit 3)
 				)
@@
 		(on_board yes)
 		(dnp no)
-		(property "Reference" "U93"
+		(property "Reference" "U50"
 			(at 895.858 506.476 0)
 			(effects
@@
 			(project ""
 				(path "/6830c6b4-6be7-4c03-9ee4-6b48bd06f260"
-					(reference "U93")
+					(reference "U50")
 					(unit 4)
 				)
@@
 		(on_board yes)
 		(dnp no)
-		(property "Reference" "U94"
+		(property "Reference" "U50"
 			(at 898.398 346.456 0)
 			(effects
@@
 			(project ""
 				(path "/6830c6b4-6be7-4c03-9ee4-6b48bd06f260"
-					(reference "U94")
+					(reference "U50")
 					(unit 2)
 				)

Commit message: Fix Tantalum capacitor footprint to use installed KiCad library
Replace non-existent Capacitor_SMD:C_Tantalum_E_7.3x4.3mm_P4.10mm with
Capacitor_Tantalum_SMD:CP_EIA-3528-21_Kemet-B (B-case 3.5x2.8mm Tantalum)
for all 10 polarized capacitors (Cp71-75, Cp91-92, Cp101, C402, C404).

https://claude.ai/code/session_01A9HsvNeuoFeWKhVBvcw39T
Parts:
- C402, C404, Cp101, Cp71, Cp72, Cp73, Cp74, Cp75, Cp91, Cp92: footprint Capacitor_SMD:C_Tantalum_E_7.3x4.3mm_P4.10mm -> Capacitor_Tantalum_SMD:CP_EIA-3528-21_Kemet-B
Changed lines of the file:
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@@
 			)
 		)
-		(property "Footprint" "Capacitor_SMD:C_Tantalum_E_7.3x4.3mm_P4.10mm"
+		(property "Footprint" "Capacitor_Tantalum_SMD:CP_EIA-3528-21_Kemet-B"
 			(at 369.57 717.55 0)
 			(effects
@@
 			)
 		)
-		(property "Footprint" "Capacitor_SMD:C_Tantalum_E_7.3x4.3mm_P4.10mm"
+		(property "Footprint" "Capacitor_Tantalum_SMD:CP_EIA-3528-21_Kemet-B"
 			(at 791.21 608.33 0)
 			(effects
@@
 			)
 		)
-		(property "Footprint" "Capacitor_SMD:C_Tantalum_E_7.3x4.3mm_P4.10mm"
+		(property "Footprint" "Capacitor_Tantalum_SMD:CP_EIA-3528-21_Kemet-B"
 			(at 463.55 720.09 0)
 			(effects
@@
 			)
 		)
-		(property "Footprint" "Capacitor_SMD:C_Tantalum_E_7.3x4.3mm_P4.10mm"
+		(property "Footprint" "Capacitor_Tantalum_SMD:CP_EIA-3528-21_Kemet-B"
 			(at 290.83 722.63 0)
 			(effects
@@
 			)
 		)
-		(property "Footprint" "Capacitor_SMD:C_Tantalum_E_7.3x4.3mm_P4.10mm"
+		(property "Footprint" "Capacitor_Tantalum_SMD:CP_EIA-3528-21_Kemet-B"
 			(at 179.07 577.85 0)
 			(effects
@@
 			)
 		)
-		(property "Footprint" "Capacitor_SMD:C_Tantalum_E_7.3x4.3mm_P4.10mm"
+		(property "Footprint" "Capacitor_Tantalum_SMD:CP_EIA-3528-21_Kemet-B"
 			(at 356.87 173.99 0)
 			(effects
@@
 			)
 		)
-		(property "Footprint" "Capacitor_SMD:C_Tantalum_E_7.3x4.3mm_P4.10mm"
+		(property "Footprint" "Capacitor_Tantalum_SMD:CP_EIA-3528-21_Kemet-B"
 			(at 422.91 120.65 0)
 			(effects
@@
 			)
 		)
-		(property "Footprint" "Capacitor_SMD:C_Tantalum_E_7.3x4.3mm_P4.10mm"
+		(property "Footprint" "Capacitor_Tantalum_SMD:CP_EIA-3528-21_Kemet-B"
 			(at 270.51 720.09 0)
 			(effects
@@
 			)
 		)
-		(property "Footprint" "Capacitor_SMD:C_Tantalum_E_7.3x4.3mm_P4.10mm"
+		(property "Footprint" "Capacitor_Tantalum_SMD:CP_EIA-3528-21_Kemet-B"
 			(at 275.59 577.85 0)
 			(effects
@@
 			)
 		)
-		(property "Footprint" "Capacitor_SMD:C_Tantalum_E_7.3x4.3mm_P4.10mm"
+		(property "Footprint" "Capacitor_Tantalum_SMD:CP_EIA-3528-21_Kemet-B"
 			(at 189.23 717.55 0)
 			(effects
